Commit message: last summit

File: my_rb1_description/src/urdf/my_rb1_robot.urdf (robot description, URDF)
Before this commit: robot rb1, 7 links, 6 joints
Links:
- removed link link_front_laser
- added link link_laser_scan, mass 0.5; collision cylinder length=0.020 radius=0.015; visual cylinder length=0.020 radius=0.015
- link base_footprint: geometry visual cylinder length=0.025 radius=0.25
- link link_left_wheel: geometry collision cylinder length=0.075 radius=0.025; visual cylinder length=0.075 radius=0.025
- link link_right_wheel: geometry collision cylinder length=0.075 radius=0.025; visual cylinder length=0.075 radius=0.025
Joints:
- removed joint joint_front_laser_base
- added joint joint_laser_scan_chassis: type fixed, parent base_link, child link_laser_scan, origin xyz=0.25 0 0.075 rpy=3.14159 0 0

Commit message: Rviz part corrected

File: my_rb1_description/src/urdf/my_rb1_robot.urdf (robot description, URDF)
Before this commit: robot rb1, 7 links, 6 joints
Links:
- link base_footprint: geometry 
- link base_link: geometry collision cylinder length=0.30 radius=0.25; visual cylinder length=0.30 radius=0.25
- link link_left_wheel: geometry collision cylinder length=0.03 radius=0.03125; visual cylinder length=0.03 radius=0.03125
- link link_right_wheel: geometry collision cylinder length=0.03 radius=0.03125; visual cylinder length=0.03 radius=0.03125
Joints:
- joint joint_chassis_left_wheel: limit effort=10000 velocity=1000 -> (none); origin xyz=0.0 0.2 -0.15 rpy=0 0 0 -> xyz=0 0.25 -0.15 rpy=0 0 0
- joint joint_chassis_right_wheel: limit effort=10000 velocity=1000 -> (none); origin xyz=0.0 -0.2 -0.15 rpy=0 0 0 -> xyz=0 -0.25 -0.15 rpy=0 0 0
